Commit message: agregado; comandos, agregado; actuador corto

File: src/my_project_pkg/model/urdf/URDFMODELFULL.urdf (robot description, URDF)
Before this commit: robot ROBOT_urdf, 7 links, 6 joints
Links:
- removed link ACTUADORFINAL1
- added link ACTUADORCORTO, mass 0.045336; collision mesh filename=package://my_project_pkg/model/meshes/ACTUADORCORTO.stl scale=0.0025 0.0025 0.0025; visual mesh filename=package://my_project_pkg/model/meshes/ACTUADORCORTO.stl scale=0.0025 0.0025 0.0025
Joints:
- removed joint ACTUADORFINAL1_joint
- added joint ACTUADORCORTO_joint: type fixed, parent CHASSISFULL, child ACTUADORCORTO, origin xyz=0 0 0.26 rpy=0 0 0, axis 0 0 -1
- joint PALASV2: parent CHASSISFULL -> ACTUADORCORTO

Commit message: carcaza+nuevas piezas

File: src/my_project_pkg/model/urdf/URDFMODELFULL.urdf (robot description, URDF)
Before this commit: robot ROBOT_urdf, 7 links, 6 joints
Links:
- added link CUERPO1, mass 0.30841; collision mesh filename=package://my_project_pkg/model/meshes/CUERPO1.stl scale=0.0025 0.0025 0.0025; visual mesh filename=package://my_project_pkg/model/meshes/CUERPO1.stl scale=0.0025 0.0025 0.0025
- added link LIDAR, mass 0.30841; collision mesh filename=package://my_project_pkg/model/meshes/LIDAR.stl scale=0.0025 0.0025 0.0025; visual mesh filename=package://my_project_pkg/model/meshes/LIDAR.stl scale=0.0025 0.0025 0.0025
- added link SOPORTE1, mass 0.30841; collision mesh filename=package://my_project_pkg/model/meshes/SOPORTE1.stl scale=0.0025 0.0025 0.0025; visual mesh filename=package://my_project_pkg/model/meshes/SOPORTE1.stl scale=0.0025 0.0025 0.0025
- added link SOPORTE2, mass 0.30841; collision mesh filename=package://my_project_pkg/model/meshes/SOPORTE2.stl scale=0.0025 0.0025 0.0025; visual mesh filename=package://my_project_pkg/model/meshes/SOPORTE2.stl scale=0.0025 0.0025 0.0025
- added link base_link; visual box size=0.01 0.01 0.01
- link CHASSISFULL: geometry collision mesh filename=/home/user/project_ws/src/my_project_pkg/model/meshes/CHASS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 scale=0.0025 0.0025 0.0025; visual mesh filename=/home/user/project_ws/src/my_project_pkg/model/meshes/CHASS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 scale=0.0025 0.0025 0.0025
Joints:
- removed joint PALASV2
- added joint CUERPO1_joint: type fixed, parent CHASSISFULL, child CUERPO1, origin xyz=0 0 0.26 rpy=0 0 0, axis 0 0 -1
- added joint LIDAR_joint: type fixed, parent CHASSISFULL, child LIDAR, origin xyz=0 0 0.26 rpy=0 0 0, axis 0 0 -1
- added joint PALASV2_joint: type prismatic, parent ACTUADORCORTO, child PALASV2, origin xyz=0 0 0.05 rpy=0 0 0, axis 0 0 1, limit lower=-0.03 upper=0.1 effort=50.0 velocity=16.0
- added joint SOPORTE1_joint: type fixed, parent CHASSISFULL, child SOPORTE1, origin xyz=0 0 0.26 rpy=0 0 0, axis 0 0 -1
- added joint SOPORTE2_joint: type fixed, parent CHASSISFULL, child SOPORTE2, origin xyz=0 0 0.26 rpy=0 0 0, axis 0 0 -1
- added joint base_to_chassis: type fixed, parent base_link, child CHASSISFULL, origin xyz=0 0 0 rpy=0 0 0
